Commit message: joint1 name adjustment

File: simplebot/urdf/backup.urdf (robot description, URDF)
Before this commit: robot simplebot, 2 links, 1 joints
Joints:
- removed joint joint_1
- added joint joint1: type continuous, parent base, child child_link, origin xyz=0 0 .2 rpy=0 0 0, axis 1 0 0

File: simplebot/urdf/simplebot.urdf (robot description, URDF)
Before this commit: robot simplebot, 3 links, 2 joints
Joints:
- removed joint joint_1
- added joint joint1: type continuous, parent base, child child_link, origin xyz=0 0 .2 rpy=0 0 0, axis 1 0 0

File: trybot_description/urdf/trybot.xacro (robot description, xacro)
@@ -116,5 +116,5 @@
     <child link="axis1"/>
   </joint>
-  <joint name="joint_1" type="prismatic">
+  <joint name="joint1" type="prismatic">
     <limit lower="-0.45" upper="0.45" effort="12" velocity="2.443"/>
   	<parent link="axis1" />
@@ -138,10 +138,10 @@
   </joint>
   <!-- ************* ACTUATOR TRANSMISSIONS ************* -->
-	<transmission name="joint_1_trans">
+	<transmission name="joint1_trans">
 		<type>transmission_interface/SimpleTransmission</type>
-		<joint name="joint_1">
+		<joint name="joint1">
 			<hardwareInterface>hardware_interface/EffortJointInterface</hardwareInterface>
 		</joint>
-		<actuator name="joint_1_motor">
+		<actuator name="joint1_motor">
 			<mechanicalReduction>1</mechanicalReduction>
 		</actuator>

Commit message: configured Rviz visualization and commander node

File: simplebot/urdf/backup.urdf (robot description, URDF)
Before this commit: robot simplebot, 2 links, 1 joints
Links:
- added link world
- link base: mass None -> 10
- link child_link: mass 0.10 -> 0.18
Joints:
- added joint worldFix: type fixed, parent world, child base

File: trybot_description/urdf/trybot.xacro (robot description, xacro)
@@ -122,5 +122,5 @@
     <axis xyz="-1 0 0" />
   </joint>
-	<joint name="joint_2" type="prismatic">
+	<joint name="joint2" type="prismatic">
     <limit lower="-0.4" upper="0.5" effort="12" velocity="2.443"/>
   	<parent link="axis2" />
@@ -129,5 +129,5 @@
     <axis xyz="0 1 0" />
   </joint>
-	<joint name="joint_3" type="prismatic">
+	<joint name="joint3" type="prismatic">
     <limit lower="-0.4" upper="0.5" effort="12" velocity="2.443"/>
   	<parent link="axis3" />
@@ -146,19 +146,19 @@
 		</actuator>
 	</transmission>
-  <transmission name="joint_2_trans">
+  <transmission name="joint2_trans">
     <type>transmission_interface/SimpleTransmission</type>
-    <joint name="joint_2">
+    <joint name="joint2">
       <hardwareInterface>hardware_interface/EffortJointInterface</hardwareInterface>
     </joint>
-    <actuator name="joint_2_motor">
+    <actuator name="joint2_motor">
       <mechanicalReduction>50</mechanicalReduction>
     </actuator>
   </transmission>
-  <transmission name="joint_3_trans">
+  <transmission name="joint3_trans">
     <type>transmission_interface/SimpleTransmission</type>
-    <joint name="joint_3">
+    <joint name="joint3">
       <hardwareInterface>hardware_interface/EffortJointInterface</hardwareInterface>
     </joint>
-    <actuator name="joint_3_motor">
+    <actuator name="joint3_motor">
       <mechanicalReduction>50</mechanicalReduction>
     </actuator>
